Commit message: model spawning works

File: versenypalya/urdf/wheel.xacro (robot description, xacro)
@@ -2,5 +2,5 @@
 <robot xmlns:xacro="http://ros.org/wiki/xacro" name="test_wheel">
 	<xacro:macro name="test_wheel" params="wheel_prefix *joint_pose">
-		<link name="${wheel_prefix}_wheel_link">
+		<link name="${wheel_prefix}">
 			<inertial>
 				<mass value="2.637" />
@@ -13,5 +13,5 @@
                     <!--cylinder length="${wheel_length}" radius="${wheel_radius}" /-->
                     <!--mesh filename = "package://urdf_examples/meshes/wheel.dae"/-->
-					<mesh filename = "package://urdf_examples/meshes/wheel_v1.dae"/>
+					<mesh filename = "package://versenypalya/meshes/wheel_v1.dae"/>
 				</geometry>
                 <material name="green"/>
@@ -24,5 +24,5 @@
 			</collision>
 		</link>
-		<gazebo reference="${wheel_prefix}_wheel_link">
+		<gazebo reference="${wheel_prefix}">
 			<mu1 value="1.0"/>
 			<mu2 value="1.0"/>
@@ -33,5 +33,5 @@
 		<joint name="${wheel_prefix}_wheel" type="continuous">
 			<parent link="base_link"/>
-			<child link="${wheel_prefix}_wheel_link"/>
+			<child link="${wheel_prefix}"/>
 			<xacro:insert_block name="joint_pose"/>
 			<axis xyz="0 1 0" rpy="0 0 0" />

File: versenypalya/urdf/xacro_test.xacro (robot description, xacro)
@@ -1,14 +1,16 @@
 <?xml version='1.0'?>
 <robot name="test_bot" xmlns:xacro="http://www.ros.org/wiki/xacro">
+  <!-- Gazebo plugin -->
+  <xacro:include filename="$(find versenypalya)/urdf/test_bot.gazebo" />
   <!-- RViz colors -->
-  <xacro:include filename="$(find urdf_examples)/urdf/materials.xacro" />
+  <xacro:include filename="$(find versenypalya)/urdf/materials.xacro" />
   <!-- Include wheel macros -->
-  <xacro:include filename="$(find urdf_examples)/urdf/wheel.xacro" />
+  <xacro:include filename="$(find versenypalya)/urdf/wheel.xacro" />
   <!-- Pi -->
   <xacro:property name="M_PI" value="3.14159"/>
   <!-- Base Size -->
-  <xacro:property name="base_x_size" value="2.285" />
-  <xacro:property name="base_y_size" value="0.806" />
-  <xacro:property name="base_z_size" value="1.369" />
+  <xacro:property name="base_x_size" value="0.2285" />
+  <xacro:property name="base_y_size" value="0.0806" />
+  <xacro:property name="base_z_size" value="0.1369" />
   <!-- Wheel Mounting Positions -->
   <xacro:property name="wheelbase" value="0.152" />
@@ -16,6 +18,6 @@
   <xacro:property name="wheel_vertical_offset" value="0.015" />
   <!-- Wheel Properties -->
-  <xacro:property name="wheel_length" value="0.296" />
-  <xacro:property name="wheel_radius" value="0.15365" />
+  <xacro:property name="wheel_length" value="0.0296" />
+  <xacro:property name="wheel_radius" value="0.015365" />
   <link name="base_footprint"></link>
   <joint name="base_footprint_joint" type="fixed">
@@ -47,5 +49,5 @@
         <!--box size="${base_x_size} ${base_y_size} ${base_z_size}"/-->
         <!--mesh filename = "package://urdf_examples/meshes/base_link.dae"/-->
-        <mesh filename = "package://urdf_examples/meshes/CarBody.dae"/>
+        <mesh filename = "package://versenypalya/meshes/CarBody.dae"/>
       </geometry>
       <material name="orange"/>
@@ -65,3 +67,52 @@
     <origin xyz="${-wheelbase/2} ${-track/2} ${wheel_vertical_offset}" rpy="0 0 0" />
   </xacro:test_wheel>
+  <!-- Camera -->
+  <joint type="fixed" name="camera_joint">
+    <origin xyz="0.225 0 0.075" rpy="0 0 0"/>
+    <child link="camera_link"/>
+    <parent link="base_link"/>
+    <axis xyz="0 1 0" />
+  </joint>
+  <link name='camera_link'>
+    <pose>0 0 0 0 0 0</pose>
+    <inertial>
+      <mass value="0.1"/>
+      <origin xyz="0 0 0" rpy="0 0 0"/>
+      <inertia
+          ixx="1e-6" ixy="0" ixz="0"
+          iyy="1e-6" iyz="0"
+          izz="1e-6"
+      />
+    </inertial>
+    <collision name='collision'>
+      <origin xyz="0 0 0" rpy="0 0 0"/>
+      <geometry>
+        <box size=".05 .05 .05"/>
+      </geometry>
+    </collision>
+    <visual name='camera_link_visual'>
+      <origin xyz="0 0 0" rpy="0 0 0"/>
+      <geometry>
+        <box size=".05 .05 .05"/>
+      </geometry>
+    </visual>
+  </link>
+  <gazebo reference="camera_link">
+    <material>Gazebo/Red</material>
+  </gazebo>
+  <joint type="fixed" name="camera_optical_joint">
+    <origin xyz="0 0 0" rpy="-1.5707 0 -1.5707"/>
+    <child link="camera_link_optical"/>
+    <parent link="camera_link"/>
+  </joint>
+  <link name="camera_link_optical">
+  </link>
+  <!-- IMU -->
+  <joint name="imu_joint" type="fixed">
+    <origin xyz="0 0 0" rpy="0 0 0" />
+    <parent link="base_link"/>
+    <child link="imu_link" />
+  </joint>
+  <link name="imu_link">
+  </link>
 </robot>

Commit message: fixed collision box, added P controller

File: versenypalya/urdf/wheel.xacro (robot description, xacro)
@@ -38,3 +38,40 @@
 		</joint>
 	</xacro:macro>
+	<xacro:macro name="test_wheel_lf" params="wheel_prefix *joint_pose">
+		<link name="${wheel_prefix}">
+			<inertial>
+				<mass value="2.637" />
+				<origin xyz="0 0 0" rpy="0 ${M_PI/2} ${M_PI/2}"/>
+				<inertia  ixx="0.02467" ixy="0" ixz="0" iyy="0.04411" iyz="0" izz="0.02467" />
+			</inertial>
+			<visual>
+				<origin xyz="0 0 0" rpy="0 ${M_PI/2} ${M_PI/2}" />
+				<geometry>
+                    <!--cylinder length="${wheel_length}" radius="${wheel_radius}" /-->
+                    <!--mesh filename = "package://urdf_examples/meshes/wheel.dae"/-->
+					<mesh filename = "package://versenypalya/meshes/wheel_v1.dae"/>
+				</geometry>
+                <material name="green"/>
+			</visual>
+			<collision>
+				<origin xyz="0 0 0" rpy="0 ${M_PI/2} ${M_PI/2}" />
+				<geometry>
+					<cylinder length="${wheel_length}" radius="${wheel_radius}" />
+				</geometry>
+			</collision>
+		</link>
+		<gazebo reference="${wheel_prefix}">
+			<mu1 value="0.0"/>
+			<mu2 value="0.0"/>
+			<kp value="0.0" />
+			<kd value="0.0" />
+			<fdir1 value="1 0 0"/>
+		</gazebo>
+		<joint name="${wheel_prefix}_wheel" type="continuous">
+			<parent link="base_link"/>
+			<child link="${wheel_prefix}"/>
+			<xacro:insert_block name="joint_pose"/>
+			<axis xyz="0 1 0" rpy="0 0 0" />
+		</joint>
+	</xacro:macro>
 </robot>

File: versenypalya/urdf/xacro_test.xacro (robot description, xacro)
@@ -12,5 +12,5 @@
   <xacro:property name="base_x_size" value="0.2285" />
   <xacro:property name="base_y_size" value="0.0806" />
-  <xacro:property name="base_z_size" value="0.1369" />
+  <xacro:property name="base_z_size" value="0.0369" />
   <!-- Wheel Mounting Positions -->
   <xacro:property name="wheelbase" value="0.152" />
@@ -39,5 +39,5 @@
     </inertial>
     <collision name='collision'>
-      <origin xyz="0 0 0" rpy="0 0 0"/>
+      <origin xyz="0 0 0.02" rpy="0 0 0"/>
       <geometry>
         <box size="${base_x_size} ${base_y_size} ${base_z_size}"/>
@@ -69,5 +69,5 @@
   <!-- Camera -->
   <joint type="fixed" name="camera_joint">
-    <origin xyz="0.225 0 0.075" rpy="0 0 0"/>
+    <origin xyz="0 0 0.075" rpy="0 0 0"/>
     <child link="camera_link"/>
     <parent link="base_link"/>

Commit message: Directory cleanup

File: versenypalya/urdf/wheel.xacro (robot description, xacro)
@@ -38,40 +38,3 @@
 		</joint>
 	</xacro:macro>
-	<xacro:macro name="test_wheel_lf" params="wheel_prefix *joint_pose">
-		<link name="${wheel_prefix}">
-			<inertial>
-				<mass value="2.637" />
-				<origin xyz="0 0 0" rpy="0 ${M_PI/2} ${M_PI/2}"/>
-				<inertia  ixx="0.02467" ixy="0" ixz="0" iyy="0.04411" iyz="0" izz="0.02467" />
-			</inertial>
-			<visual>
-				<origin xyz="0 0 0" rpy="0 ${M_PI/2} ${M_PI/2}" />
-				<geometry>
-                    <!--cylinder length="${wheel_length}" radius="${wheel_radius}" /-->
-                    <!--mesh filename = "package://urdf_examples/meshes/wheel.dae"/-->
-					<mesh filename = "package://versenypalya/meshes/wheel_v1.dae"/>
-				</geometry>
-                <material name="green"/>
-			</visual>
-			<collision>
-				<origin xyz="0 0 0" rpy="0 ${M_PI/2} ${M_PI/2}" />
-				<geometry>
-					<cylinder length="${wheel_length}" radius="${wheel_radius}" />
-				</geometry>
-			</collision>
-		</link>
-		<gazebo reference="${wheel_prefix}">
-			<mu1 value="0.0"/>
-			<mu2 value="0.0"/>
-			<kp value="0.0" />
-			<kd value="0.0" />
-			<fdir1 value="1 0 0"/>
-		</gazebo>
-		<joint name="${wheel_prefix}_wheel" type="continuous">
-			<parent link="base_link"/>
-			<child link="${wheel_prefix}"/>
-			<xacro:insert_block name="joint_pose"/>
-			<axis xyz="0 1 0" rpy="0 0 0" />
-		</joint>
-	</xacro:macro>
 </robot>

File: versenypalya/urdf/xacro_test.xacro (robot description, xacro)
@@ -88,5 +88,5 @@
       <origin xyz="0 0 0" rpy="0 0 0"/>
       <geometry>
-        <box size=".05 .05 .05"/>
+        <box size=".0005 .0005 .0005"/>
       </geometry>
     </collision>
@@ -94,5 +94,5 @@
       <origin xyz="0 0 0" rpy="0 0 0"/>
       <geometry>
-        <box size=".05 .05 .05"/>
+        <box size=".0005 .0005 .0005"/>
       </geometry>
     </visual>
